File: hardware/Geckoconsole.kicad_sch (KiCad schematic)
At the start: 61 parts, among them J1 Conn_01x06_Male, J11 Conn_01x06_Female, J31 Conn_01x07_Female, J50 USB-C, J51 Conn_01x06_Male, J70 I²C, J81 Conn_01x07, Q51 S8050, Q52 S8050, SW1 Reset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

Commit message: Hardware Console: Fix Encoder button (missing GND wire)
Connections:
- net GND: now also C43.2, SW41.S2
Changed lines of the file:
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@@
   (junction (at 118.11 36.83) (diameter 0) (color 0 0 0 0)
+  )
+  (junction (at 251.46 64.77) (diameter 0) (color 0 0 0 0)
   )
   (junction (at 92.71 180.34) (diameter 0) (color 0 0 0 0)
@@
     (stroke (width 0) (type default) (color 0 0 0 0))
   )
+  (wire (pts (xy 251.46 68.58) (xy 264.16 68.58))
+    (stroke (width 0) (type default) (color 0 0 0 0))
+  )
   (wire (pts (xy 83.82 180.34) (xy 83.82 187.96))
     (stroke (width 0) (type default) (color 0 0 0 0))
@@
     (stroke (width 0) (type default) (color 0 0 0 0))
   )
+  (wire (pts (xy 251.46 64.77) (xy 251.46 68.58))
+    (stroke (width 0) (type default) (color 0 0 0 0))
+  )

Commit message: Hardware Console: Use new FUET Buzzer in schematic and PCB
Parts:
- BZ1: value Buzzer -> (none); footprint Buzzer_Beeper:Buzzer_Murata_PKMCS0909E4000-R1 -> (none)
Changed lines of the file:
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@@
       (effects (font (size 1.27 1.27)) (justify right))
     )
-    (property "Value" "Buzzer" (id 1) (at 188.8998 58.166 90)
-      (effects (font (size 1.27 1.27)) (justify right))
-    )
-    (property "Footprint" "Buzzer_Beeper:Buzzer_Murata_PKMCS0909E4000-R1" (id 2) (at 181.61 57.785 90)
+    (property "Value" "" (id 1) (at 188.8998 58.166 90)
+      (effects (font (size 1.27 1.27)) (justify right))
+    )
+    (property "Footprint" "" (id 2) (at 181.61 57.785 90)
       (effects (font (size 1.27 1.27)) hide)
     )
@@
     )
     (path "/00000000-0000-0000-0000-0000610658bc"
-      (reference "BZ1") (unit 1) (value "Buzzer") (footprint "Buzzer_Beeper:Buzzer_Murata_PKMCS0909E4000-R1")
+      (reference "BZ1") (unit 1) (value "Buzzer") (footprint "Fraxinas:Buzzer_FUET_9650B")
     )
     (path "/00000000-0000-0000-0000-0000626bef05"
